Commit message: REL: moving with ZED

File: wheelchair_src/src/wheelchair_description/urdf/wheelchair.xacro (robot description, xacro)
@@ -188,3 +188,16 @@
   <axis xyz="0.0 1.0 0.0"/>
 </joint>
+ <xacro:arg name="camera_name"   default="zed" />
+  <xacro:arg name="camera_model"  default="zed" />
+  <xacro:arg name="base_frame"    default="base_link" />
+  <xacro:arg name="cam_pos_x"     default="-0.63" />
+  <xacro:arg name="cam_pos_y"     default="0.25" />
+  <xacro:arg name="cam_pos_z"     default="1.30" />
+  <xacro:arg name="cam_roll"      default="0.0" />
+  <xacro:arg name="cam_pitch"     default="0.0" />
+  <xacro:arg name="cam_yaw"       default="0.0" />
+  <xacro:include filename="$(find zed_wrapper)/urdf/zed_macro.urdf.xacro" />
+  <xacro:zed_camera name="$(arg camera_name)" model="$(arg camera_model)" parent="$(arg base_frame)">
+    <origin xyz="$(arg cam_pos_x) $(arg cam_pos_y) $(arg cam_pos_z)" rpy="$(arg cam_roll) $(arg cam_pitch) $(arg cam_yaw)" />
+  </xacro:zed_camera>
 </robot>
